File: FPGA.kicad_sch (KiCad schematic)
At the start: 0 parts

Commit message: add
Other:
- added sheet adc (adc.kicad_sch)
Changed lines of the file:
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@@
 	(sheet
 		(at 54.61 86.36)
-		(size 43.18 22.86)
+		(size 24.13 22.86)
 		(exclude_from_sim no)
 		(in_bom yes)
@@
 	)
 	(sheet
-		(at 119.38 88.9)
+		(at 95.25 86.36)
 		(size 24.13 20.32)
 		(exclude_from_sim no)
@@
 		)
 		(property "Sheetname" "FTDI"
-			(at 119.38 88.1884 0)
+			(at 95.25 85.6484 0)
 			(effects
 				(font
@@
 		)
 		(property "Sheetfile" "FTDI.kicad_sch"
-			(at 119.38 109.8046 0)
+			(at 95.25 107.2646 0)
 			(effects
 				(font
@@
 				)
 			)
+		)
+	)
+	(sheet
+		(at 139.7 81.28)
+		(size 31.75 25.4)
+		(exclude_from_sim no)
+		(in_bom yes)
+		(on_board yes)
+		(dnp no)
+		(fields_autoplaced yes)
+		(stroke
+			(width 0.1524)
+			(type solid)
+		)
+		(fill
+			(color 0 0 0 0.0000)
+		)
+		(property "Sheetname" "adc"
+			(at 139.7 80.5684 0)
+			(effects
+				(font
+					(size 1.27 1.27)
+				)
+				(justify left bottom)
+			)
+		)
+		(property "Sheetfile" "adc.kicad_sch"
+			(at 139.7 107.2646 0)
+			(effects
+				(font
+					(size 1.27 1.27)
+				)
+				(justify left top)
+			)
+		)
+		(instances
+			(project "risetRadar"
+				(path "/de705012-f0fb-4b23-929c-98742aa6def5/9ebb199d-5c8b-41dd-b601-8f5ebc1c419e"
+					(page "9")
+				)
+			)
