File: FPGA_power.kicad_sch (KiCad schematic)
At the start: 15 parts, among them U1 XC7A35T-FTG256

Commit message: add
Parts:
- added C84, C85: 0.47uF, Capacitor_SMD:C_0201_0603Metric, symbol Device:C_US
- added FB1, FB2: HZ0805E601R-10, symbol Device:FerriteBead
Connections:
- net GNDREF: now also C84.2, C85.2, FB2.2
- net VCC1V8: now also C85.1, FB1.1
- new net GNDA: FB2.1
- new net VCCA1V8: C84.1, FB1.2
Other:
- moved on the sheet: C14, C15
